File: sofle-choc-pro.kicad_sch (KiCad schematic)
At the start: 36 parts, among them J1 Connector, USB-TYPE-C-16P, J2 Connector, USB-TYPE-C-16P, SW1 SW_Push, U1 AP2112K-3.3, U1 RP2040, U2 SRV05-4A, U3 W25Q128, U4 SRV05-4A, X1 X322512MSB4SI

Commit message: feat(schematic): fix RP2040 controller and add the full keyboard half
Fixes the controller defects that would have stopped the board working and adds the matrix, LEDs, encoders and display support, audited against the RP2040 datasheet, the RP2040 hardware design guide and each part's datasheet.

- USB D+/D- now reach the RP2040 through one ESD channel each; QSPI SD0/SD1 no longer swapped; duplicate U1 renamed U5
- crystal is the reference ABM8-272-T3 with 15 pF load caps; RUN follows the minimal design (no capacitor)
- Schottky after the fuse stops two hosts back-feeding through the link; GP13 VBUS sense divider sized for the fault-tolerant pin limit
- 37-key matrix on Keebart's pin map plus F-row, extra column and second encoder, with two Choc/EC11 combo positions
- 37 SK6812MINI-E LEDs behind an SN74LV1T34 level shifter and 470 ohm series resistor
- 5-pin display header for a 128x32 OLED (I2C0) or nice!view (SPI1), selected by solder jumpers; handedness jumper and reset button
- every assembled part has a verified in-stock LCSC number; hand-soldered parts are excluded from the BOM
Parts:
- removed C21: 100nF, PCM_JLCPCB:C_0402, symbol PCM_JLCPCB-Capacitors:0402,100nF
- added C110, C111, C112, C113, C114, C115, C116, C120, C121, C122, C123, C124, C125, C130, C131, C132, C133, C134, C135, C140, C141, C142, C143, C144, C145, C150, C151, C152, C153, C154, C155, C160, C161, C162, C163, C164, C165, C30: 100nF, PCM_JLCPCB:C_0402, symbol PCM_JLCPCB-Capacitors:0402,100nF
- added D1: B5819W SL, PCM_JLCPCB:D_SOD-123, symbol PCM_JLCPCB-Diodes:Schottky,B5819W SL
- added D10, D11, D12, D13, D14, D15, D16, D20, D21, D22, D23, D24, D25, D30, D31, D32, D33, D34, D35, D40, D41, D42, D43, D44, D45, D50, D51, D52, D53, D54, D55, D60, D61, D62, D63, D64, D65: 1N4148W, PCM_JLCPCB:D_SOD-123, symbol PCM_JLCPCB-Diodes:Switching,1N4148W
- added J3: OLED 128x32 / nice!view, Connector_PinHeader_2.54mm:PinHeader_1x05_P2.54mm_Vertical, symbol Connector_Generic:Conn_01x05
- added JP1: HAND L=1-2 R=2-3, Jumper:SolderJumper-3_P1.3mm_Open_RoundedPad1.0x1.5mm_NumberLabels, symbol Jumper:SolderJumper_3_Open
- added JP2: SCL OLED=1-2 VIEW=2-3, Jumper:SolderJumper-3_P1.3mm_Open_RoundedPad1.0x1.5mm_NumberLabels, symbol Jumper:SolderJumper_3_Open
- added JP3: SDA OLED=1-2 VIEW=2-3, Jumper:SolderJumper-3_P1.3mm_Open_RoundedPad1.0x1.5mm_NumberLabels, symbol Jumper:SolderJumper_3_Open
- added LED10, LED11, LED12, LED13, LED14, LED15, LED16, LED20, LED21, LED22, LED23, LED24, LED25, LED30, LED31, LED32, LED33, LED34, LED35, LED40, LED41, LED42, LED43, LED44, LED45, LED50, LED51, LED52, LED53, LED54, LED55, LED60, LED61, LED62, LED63, LED64, LED65: SK6812MINI-E, my-soffle:LED-SMD_4P-L3.2-W2.8-LS5.9_SK6812MINI-E, symbol my-soffle:SK6812MINI-E_C5149201
- added R10: 10kΩ, PCM_JLCPCB:R_0402, symbol PCM_JLCPCB-Resistors:0402,10kΩ
- added R11: 15kΩ, PCM_JLCPCB:R_0402, symbol PCM_JLCPCB-Resistors:0402,15kΩ
- added R12, R13: 4.7kΩ, PCM_JLCPCB:R_0402, symbol PCM_JLCPCB-Resistors:0402,4.7kΩ
- added R15: 470Ω, PCM_JLCPCB:R_0402, symbol PCM_JLCPCB-Resistors:0402,470Ω
- added SW10: F0, my-soffle:SW_Choc_V1V2_Hotswap_1.00u, symbol Switch:SW_Push
- added SW11: F1, my-soffle:SW_Choc_V1V2_Hotswap_1.00u, symbol Switch:SW_Push
- added SW12: F2, my-soffle:SW_Choc_V1V2_Hotswap_1.00u, symbol Switch:SW_Push
- added SW13: F3, my-soffle:SW_Choc_V1V2_Hotswap_1.00u, symbol Switch:SW_Push
- added SW14: F4, my-soffle:SW_Choc_V1V2_Hotswap_1.00u, symbol Switch:SW_Push
- added SW15: F5, my-soffle:SW_Choc_V1V2_Hotswap_1.00u, symbol Switch:SW_Push
- added SW16: F6 Choc/EC11, my-soffle:SW_Choc_V1V2_Hotswap_EC11_Combo, symbol my-soffle:SW_Choc_EC11_Combo
- added SW2: RESET, my-soffle:SW_Push_1P1T_XKB_TS-1187A, symbol Switch:SW_Push
- added SW20: N0, my-soffle:SW_Choc_V1V2_Hotswap_1.00u, symbol Switch:SW_Push
- added SW21: N1, my-soffle:SW_Choc_V1V2_Hotswap_1.00u, symbol Switch:SW_Push
- added SW22: N2, my-soffle:SW_Choc_V1V2_Hotswap_1.00u, symbol Switch:SW_Push
- added SW23: N3, my-soffle:SW_Choc_V1V2_Hotswap_1.00u, symbol Switch:SW_Push
- added SW24: N4, my-soffle:SW_Choc_V1V2_Hotswap_1.00u, symbol Switch:SW_Push
- added SW25: N5, my-soffle:SW_Choc_V1V2_Hotswap_1.00u, symbol Switch:SW_Push
- added SW30: T0, my-soffle:SW_Choc_V1V2_Hotswap_1.00u, symbol Switch:SW_Push
- added SW31: T1, my-soffle:SW_Choc_V1V2_Hotswap_1.00u, symbol Switch:SW_Push
- added SW32: T2, my-soffle:SW_Choc_V1V2_Hotswap_1.00u, symbol Switch:SW_Push
- added SW33: T3, my-soffle:SW_Choc_V1V2_Hotswap_1.00u, symbol Switch:SW_Push
- added SW34: T4, my-soffle:SW_Choc_V1V2_Hotswap_1.00u, symbol Switch:SW_Push
- added SW35: T5, my-soffle:SW_Choc_V1V2_Hotswap_1.00u, symbol Switch:SW_Push
- added SW40: H0, my-soffle:SW_Choc_V1V2_Hotswap_1.00u, symbol Switch:SW_Push
- added SW41: H1, my-soffle:SW_Choc_V1V2_Hotswap_1.00u, symbol Switch:SW_Push
- added SW42: H2, my-soffle:SW_Choc_V1V2_Hotswap_1.00u, symbol Switch:SW_Push
- added SW43: H3, my-soffle:SW_Choc_V1V2_Hotswap_1.00u, symbol Switch:SW_Push
- added SW44: H4, my-soffle:SW_Choc_V1V2_Hotswap_1.00u, symbol Switch:SW_Push
- added SW45: H5, my-soffle:SW_Choc_V1V2_Hotswap_1.00u, symbol Switch:SW_Push
- added SW50: B0, my-soffle:SW_Choc_V1V2_Hotswap_1.00u, symbol Switch:SW_Push
- added SW51: B1, my-soffle:SW_Choc_V1V2_Hotswap_1.00u, symbol Switch:SW_Push
- added SW52: B2, my-soffle:SW_Choc_V1V2_Hotswap_1.00u, symbol Switch:SW_Push
- added SW53: B3, my-soffle:SW_Choc_V1V2_Hotswap_1.00u, symbol Switch:SW_Push
- added SW54: B4, my-soffle:SW_Choc_V1V2_Hotswap_1.00u, symbol Switch:SW_Push
- added SW55: B5, my-soffle:SW_Choc_V1V2_Hotswap_1.00u, symbol Switch:SW_Push
- added SW60: TH0, my-soffle:SW_Choc_V1V2_Hotswap_1.00u, symbol Switch:SW_Push
- added SW61: TH1, my-soffle:SW_Choc_V1V2_Hotswap_1.00u, symbol Switch:SW_Push
- added SW62: TH2, my-soffle:SW_Choc_V1V2_Hotswap_1.00u, symbol Switch:SW_Push
- added SW63: TH3, my-soffle:SW_Choc_V1V2_Hotswap_1.00u, symbol Switch:SW_Push
- added SW64: TH4, my-soffle:SW_Choc_V1V2_Hotswap_1.50u, symbol Switch:SW_Push
- added SW65: TH5 Choc/EC11, my-soffle:SW_Choc_V1V2_Hotswap_EC11_Combo, symbol my-soffle:SW_Choc_EC11_Combo
- added U6: SN74LV1T34DBVR, Package_TO_SOT_SMD:SOT-23-5, symbol 74xGxx:74LVC1G34
- C18: value 100uF -> 10uF; footprint PCM_JLCPCB:C_1206 -> PCM_JLCPCB:C_0603; symbol PCM_JLCPCB-Capacitors:1206,100uF -> PCM_JLCPCB-Capacitors:0603,10uF; LCSC C883598 -> C19702; Manufacturer Murata -> Samsung Electro-Mechanics; Part GRM31CR61A107MEA8L -> CL10A106KP8NNNC
- F1: footprint PCM_JLCPCB:C_1206 -> Fuse:Fuse_1206_3216Metric; LCSC C261952 -> C163512; Manufacturer TLC Electronic -> Littelfuse; Part TLC-NSMD050 -> 1206L050YR
- R5, R6: symbol PCM_JLCPCB-Resistors:0402,1.5kΩ -> PCM_JLCPCB-Resistors:0402,5.1kΩ; LCSC C23186 -> C25905; Part 0603WAF5101T5E -> 0402WGF5101TCE
- R7, R8: LCSC C352446 -> C25100
- SW1: value SW_Push -> BOOT; footprint Button_Switch_SMD:SW_Push_1P1T_XKB_TS-1187A -> my-soffle:SW_Push_1P1T_XKB_TS-1187A
- U2, U4: value SRV05-4A -> SRV05-4; Attrition Qty 4 -> (none); LCSC C20615829 -> C2836319; Manufacturer hongjiacheng -> MSKSEMI; Minimum Qty 5 -> (none); Part SRV05-4A -> SRV05-4; Price 0.048USD -> (none); Stock 68123 -> (none)
- X1: value X322512MSB4SI -> ABM8-272-T3; Attrition Qty 4 -> (none); Class Basic Component -> (none); Frequency Tolerance ±10ppm -> ±30ppm; LCSC C9002 -> C20625731; Load Capacitance 20pF -> 10pF; Manufacturer Yangxing Tech -> Abracon LLC; Minimum Qty 5 -> (none); Part X322512MSB4SI -> ABM8-272-T3; Price 0.068USD -> (none); Stock 260231 -> (none)
- renumbered U1 to U5
Connections:
- net +3.3V: now also J3.3 (Pin_3), JP1.1 (A), R12.1, R13.1; no longer C18.1
- net +5V: now also C18.1, C110.1, C111.1, C112.1, C113.1, C114.1, C115.1, C116.1, C120.1, C121.1, C122.1, C123.1, C124.1, C125.1, C130.1, C131.1, C132.1, C133.1, C134.1, C135.1, C140.1, C141.1, C142.1, C143.1, C144.1, C145.1, C150.1, C151.1, C152.1, C153.1, C154.1, C155.1, C160.1, C161.1, C162.1, C163.1, C164.1, C165.1, C30.1, D1.1, LED10.3 (VDD), LED11.3 (VDD), LED12.3 (VDD), LED13.3 (VDD), LED14.3 (VDD), LED15.3 (VDD), LED16.3 (VDD), LED20.3 (VDD), LED21.3 (VDD), LED22.3 (VDD), LED23.3 (VDD), LED24.3 (VDD), LED25.3 (VDD), LED30.3 (VDD), LED31.3 (VDD), LED32.3 (VDD), LED33.3 (VDD), LED34.3 (VDD), LED35.3 (VDD), LED40.3 (VDD), LED41.3 (VDD), LED42.3 (VDD), LED43.3 (VDD), LED44.3 (VDD), LED45.3 (VDD), LED50.3 (VDD), LED51.3 (VDD), LED52.3 (VDD), LED53.3 (VDD), LED54.3 (VDD), LED55.3 (VDD), LED60.3 (VDD), LED61.3 (VDD), LED62.3 (VDD), LED63.3 (VDD), LED64.3 (VDD), LED65.3 (VDD), U6.5 (VCC); no longer F1.2
- net D_USB_N: now also R8.1
- net D_USB_P: now also R7.1
- net GND: now also C110.2, C111.2, C112.2, C113.2, C114.2, C115.2, C116.2, C120.2, C121.2, C122.2, C123.2, C124.2, C125.2, C130.2, C131.2, C132.2, C133.2, C134.2, C135.2, C140.2, C141.2, C142.2, C143.2, C144.2, C145.2, C150.2, C151.2, C152.2, C153.2, C154.2, C155.2, C160.2, C161.2, C162.2, C163.2, C164.2, C165.2, C30.2, J3.2 (Pin_2), JP1.3 (B), LED10.1 (GND), LED11.1 (GND), LED12.1 (GND), LED13.1 (GND), LED14.1 (GND), LED15.1 (GND), LED16.1 (GND), LED20.1 (GND), LED21.1 (GND), LED22.1 (GND), LED23.1 (GND), LED24.1 (GND), LED25.1 (GND), LED30.1 (GND), LED31.1 (GND), LED32.1 (GND), LED33.1 (GND), LED34.1 (GND), LED35.1 (GND), LED40.1 (GND), LED41.1 (GND), LED42.1 (GND), LED43.1 (GND), LED44.1 (GND), LED45.1 (GND), LED50.1 (GND), LED51.1 (GND), LED52.1 (GND), LED53.1 (GND), LED54.1 (GND), LED55.1 (GND), LED60.1 (GND), LED61.1 (GND), LED62.1 (GND), LED63.1 (GND), LED64.1 (GND), LED65.1 (GND), R11.2, SW16.C, SW2.1, SW65.C, U6.3 (GND)
- net GP12: now also J2.A6 (D+), J2.B6 (D+)
- net GP21: now also JP1.2 (C); no longer U2.3 (I/O)
- net SD0: now also U3.5 (DI); no longer U3.2 (DO)
- net SD1: now also U3.2 (DO); no longer U3.5 (DI)
- net VBUS: now also R10.1
- net RUN: now reaches U1.26 (RUN)
- net RUN: now also SW2.2
- net GP8: now reaches U1.11 (GPIO8)
- net GP8: now also SW16.B
- net GP10: now reaches U1.13 (GPIO10)
- net GP10: now also U6.2
- net GP11: now reaches U1.14 (GPIO11)
- net GP11: now also J3.1 (Pin_1)
- net GP13: now reaches U1.16 (GPIO13)
- net GP13: now also R10.2, R11.1
- net GP14: now reaches U1.17 (GPIO14)
- net GP14: now also JP2.3 (B)
- net GP15: now reaches U1.18 (GPIO15)
- net GP15: now also JP3.3 (B)
- net GP0: now reaches U1.2 (GPIO0)
- net GP0: now also D20.1, D21.1, D22.1, D23.1, D24.1, D25.1
- net GP18: now reaches U1.29 (GPIO18)
- net GP18: now also SW15.1, SW25.1, SW35.1, SW45.1, SW55.1, SW65.1 (SW)
- net GP1: now reaches U1.3 (GPIO1)
- net GP1: now also D30.1, D31.1, D32.1, D33.1, D34.1, D35.1
- net GP19: now reaches U1.30 (GPIO19)
- net GP19: now also SW14.1, SW24.1, SW34.1, SW44.1, SW54.1, SW64.1
- net GP22: now reaches U1.34 (GPIO22)
- net GP22: now also SW65.B
- net GP23: now reaches U1.35 (GPIO23)
- net GP23: now also SW65.A
- net GP24: now reaches U1.36 (GPIO24)
- net GP24: now also SW13.1, SW23.1, SW33.1, SW43.1, SW53.1, SW63.1
- net GP25: now reaches U1.37 (GPIO25)
- net GP25: now also SW12.1, SW22.1, SW32.1, SW42.1, SW52.1, SW62.1
- net GP26: now reaches U1.38 (GPIO26_ADC0)
- net GP26: now also SW11.1, SW21.1, SW31.1, SW41.1, SW51.1, SW61.1
- net GP27: now reaches U1.39 (GPIO27_ADC1)
- net GP27: now also SW10.1, SW20.1, SW30.1, SW40.1, SW50.1, SW60.1
- net GP2: now reaches U1.4 (GPIO2)
- net GP2: now also D40.1, D41.1, D42.1, D43.1, D44.1, D45.1
- net GP28: now reaches U1.40 (GPIO28_ADC2)
- net GP28: now also JP3.1 (A), R12.2
- net GP29: now reaches U1.41 (GPIO29_ADC3)
- net GP29: now also JP2.1 (A), R13.2
- net GP3: now reaches U1.5 (GPIO3)
- net GP3: now also D50.1, D51.1, D52.1, D53.1, D54.1, D55.1
- net GP4: now reaches U1.6 (GPIO4)
- net GP4: now also D60.1, D61.1, D62.1, D63.1, D64.1, D65.1
- net GP5: now reaches U1.7 (GPIO5)
- net GP5: now also SW16.1 (SW)
- net GP6: now reaches U1.8 (GPIO6)
- net GP6: now also D10.1, D11.1, D12.1, D13.1, D14.1, D15.1, D16.1
- net GP7: now reaches U1.9 (GPIO7)
- net GP7: now also SW16.A
- net D_N: no longer names the net of U4.4 (I/O)
- net D_N: no longer R8.1
- net D_P: no longer names the net of U4.3 (I/O)
- net D_P: no longer R7.1
- removed net SPLIT_D_P: J2.A6 (D+), J2.B6 (D+), U2.6 (I/O)
- new net: D43.2, SW43.2
- new net: D1.2, F1.2
- new net: D54.2, SW54.2
- new net: D16.2, SW16.2 (SW)
- new net: D12.2, SW12.2
- new net: D44.2, SW44.2
- new net: D55.2, SW55.2
- new net: D35.2, SW35.2
- new net: D20.2, SW20.2
- new net: D34.2, SW34.2
- new net: D22.2, SW22.2
- new net: D21.2, SW21.2
- new net: D10.2, SW10.2
- new net: D65.2, SW65.2 (SW)
- new net: D64.2, SW64.2
- new net: D63.2, SW63.2
- new net: D24.2, SW24.2
- new net: D53.2, SW53.2
- new net: D25.2, SW25.2
- new net: D52.2, SW52.2
- new net: D51.2, SW51.2
- new net: D62.2, SW62.2
- new net: D33.2, SW33.2
- new net: D40.2, SW40.2
- new net: D61.2, SW61.2
- new net: D41.2, SW41.2
- new net: D45.2, SW45.2
- new net: D50.2, SW50.2
- new net: D60.2, SW60.2
- new net: D15.2, SW15.2
- new net: D32.2, SW32.2
- new net: D14.2, SW14.2
- new net: D13.2, SW13.2
- new net: D23.2, SW23.2
- new net: D42.2, SW42.2
- new net: D31.2, SW31.2
- new net: D11.2, SW11.2
- new net: D30.2, SW30.2
- new net DISP_SCL: J3.4 (Pin_4), JP2.2 (C)
- new net DISP_SDA: J3.5 (Pin_5), JP3.2 (C)
- new net LED_BUF: R15.1, U6.4
- new net LED_D0: LED65.2 (DIN), R15.2
- new net LED_D1: LED64.2 (DIN), LED65.4 (DOUT)
- new net LED_D10: LED14.4 (DOUT), LED24.2 (DIN)
- new net LED_D11: LED24.4 (DOUT), LED34.2 (DIN)
- new net LED_D12: LED34.4 (DOUT), LED44.2 (DIN)
- new net LED_D13: LED44.4 (DOUT), LED54.2 (DIN)
- new net LED_D14: LED54.4 (DOUT), LED62.2 (DIN)
- new net LED_D15: LED61.2 (DIN), LED62.4 (DOUT)
- new net LED_D16: LED53.2 (DIN), LED61.4 (DOUT)
- new net LED_D17: LED43.2 (DIN), LED53.4 (DOUT)
- new net LED_D18: LED33.2 (DIN), LED43.4 (DOUT)
- new net LED_D19: LED23.2 (DIN), LED33.4 (DOUT)
- new net LED_D2: LED63.2 (DIN), LED64.4 (DOUT)
- new net LED_D20: LED13.2 (DIN), LED23.4 (DOUT)
- new net LED_D21: LED12.2 (DIN), LED13.4 (DOUT)
- new net LED_D22: LED12.4 (DOUT), LED22.2 (DIN)
- new net LED_D23: LED22.4 (DOUT), LED32.2 (DIN)
- new net LED_D24: LED32.4 (DOUT), LED42.2 (DIN)
- new net LED_D25: LED42.4 (DOUT), LED52.2 (DIN)
- new net LED_D26: LED52.4 (DOUT), LED60.2 (DIN)
- new net LED_D27: LED51.2 (DIN), LED60.4 (DOUT)
- new net LED_D28: LED41.2 (DIN), LED51.4 (DOUT)
- new net LED_D29: LED31.2 (DIN), LED41.4 (DOUT)
- new net LED_D3: LED55.2 (DIN), LED63.4 (DOUT)
- new net LED_D30: LED21.2 (DIN), LED31.4 (DOUT)
- new net LED_D31: LED11.2 (DIN), LED21.4 (DOUT)
- new net LED_D32: LED10.2 (DIN), LED11.4 (DOUT)
- new net LED_D33: LED10.4 (DOUT), LED20.2 (DIN)
- new net LED_D34: LED20.4 (DOUT), LED30.2 (DIN)
- new net LED_D35: LED30.4 (DOUT), LED40.2 (DIN)
- new net LED_D36: LED40.4 (DOUT), LED50.2 (DIN)
- new net LED_D4: LED45.2 (DIN), LED55.4 (DOUT)
- new net LED_D5: LED35.2 (DIN), LED45.4 (DOUT)
- new net LED_D6: LED25.2 (DIN), LED35.4 (DOUT)
- new net LED_D7: LED15.2 (DIN), LED25.4 (DOUT)
- new net LED_D8: LED15.4 (DOUT), LED16.2 (DIN)
- new net LED_D9: LED14.2 (DIN), LED16.4 (DOUT)
- no-connect marks 12 -> 18

Commit message: feat(pcb): use 2-pin ts-1088 buttons for boot and reset
BOOT and RESET (SW1, SW2) now use the smaller 2-terminal XUNPU
TS-1088-AR02016 tactile switch instead of the 4-pin TS-1187A.

- LCSC C720477 is a JLCPCB Basic part, so no extended-part fee
- 4 x 3 mm body with one pad per short end, easier to fit and route
- Footprint and STEP model live in the project library, so the board
  does not depend on the PCM JLCPCB library being installed

Swapped in place: same position, side, rotation and nets. ERC 0 errors;
DRC counts did not rise and schematic parity passes.
Parts:
- SW1, SW2: footprint my-soffle:SW_Push_1P1T_XKB_TS-1187A -> my-soffle:SW_Push_1P1T_XUNPU_TS-1088-AR02016; LCSC C318884 -> C720477; Part TS-1187A-B-A-B -> TS-1088-AR02016
Changed lines of the file:
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@@
 			)
 		)
-		(property "Footprint" "my-soffle:SW_Push_1P1T_XKB_TS-1187A"
+		(property "Footprint" "my-soffle:SW_Push_1P1T_XUNPU_TS-1088-AR02016"
 			(at 24.13 161.29 0)
 			(hide yes)
@@
 			)
 		)
-		(property "LCSC" "C318884"
+		(property "LCSC" "C720477"
 			(at 24.13 166.37 0)
 			(hide yes)
@@
 			)
 		)
-		(property "Part" "TS-1187A-B-A-B"
+		(property "Part" "TS-1088-AR02016"
 			(at 24.13 166.37 0)
 			(hide yes)
@@
 			)
 		)
-		(property "Footprint" "my-soffle:SW_Push_1P1T_XKB_TS-1187A"
+		(property "Footprint" "my-soffle:SW_Push_1P1T_XUNPU_TS-1088-AR02016"
 			(at 254 86.36 0)
 			(hide yes)
@@
 			)
 		)
-		(property "LCSC" "C318884"
+		(property "LCSC" "C720477"
 			(at 254 86.36 0)
 			(hide yes)
@@
 			)
 		)
-		(property "Part" "TS-1187A-B-A-B"
+		(property "Part" "TS-1088-AR02016"
 			(at 254 86.36 0)
 			(hide yes)

Commit message: feat(sch): protect the link port and harden master detection
The link USB-C port could back-feed 5 V into a misplugged device and its
data line had no current limit, and diode leakage could fool the VBUS
divider on the secondary half. These fixes follow the reference boards
with a real USB-C link (Djinn, YAEMK) and Splinky's detect divider.

- F2 polyfuse (same part as F1) between J2 VBUS and +5V; the connector
  side is now LINK_VBUS, and J2 CC stays open so hosts keep VBUS off
- R16 120 ohm between J2/U2 and GP12 (net LINK_DATA on the connector
  side) limits ESD clamp current and damps cable ringing
- R10/R11 now 5.1k/10k (was 10k/15k): same 3.3 V at GP13 with a stiffer
  divider against D1 reverse leakage
- HOST and LINK labels on the back silkscreen next to J1 and J2

ERC 0 errors. DRC with schematic parity: only starved_thermal and the
expected unconnected items (board still unrouted).
Parts:
- added F2: 500mA, Fuse:Fuse_1206_3216Metric, symbol Device:Polyfuse
- added R16: 120Ω, PCM_JLCPCB:R_0402, symbol PCM_JLCPCB-Resistors:0402,120Ω
- R10: value 10kΩ -> 5.1kΩ; symbol PCM_JLCPCB-Resistors:0402,10kΩ -> PCM_JLCPCB-Resistors:0402,5.1kΩ; LCSC C25744 -> C25905; Part 0402WGF1002TCE -> 0402WGF5101TCE; Resistance 10kΩ -> 5.1kΩ
- R11: value 15kΩ -> 10kΩ; symbol PCM_JLCPCB-Resistors:0402,15kΩ -> PCM_JLCPCB-Resistors:0402,10kΩ; LCSC C25756 -> C25744; Part 0402WGF1502TCE -> 0402WGF1002TCE; Resistance 15kΩ -> 10kΩ; Stock 671055 -> 24372091
Connections:
- net +5V: now also F2.2; no longer J2.A9B4 (VBUS), J2.B9A4 (VBUS)
- net GP12: now also R16.2; no longer J2.A6 (D+), J2.B6 (D+), U2.1 (I/O)
- new net LINK_DATA: J2.A6 (D+), J2.B6 (D+), R16.1, U2.1 (I/O)
- new net LINK_VBUS: F2.1, J2.A9B4 (VBUS), J2.B9A4 (VBUS)

Commit message: feat(sch): move the matrix onto the rp2040 side facing the keys
All six rows sat on GP0-GP6, on the far side of the RP2040 from the key
block, so every row wire had to cross the package before reaching the
matrix. The matrix now uses pins 29-41, which face the keys, in the
order the bundle peels off.

- Rows 1-6 (top to thumbs) on GP29-GP24, columns 0-5 (outer to inner)
  on GP18-GP23; the encoder-key column stays on GP5
- Second encoder moves to GP3/GP4, handedness JP1 to GP2, and the
  display I2C option to GP16 (SDA) / GP17 (SCL), still I2C0
- GP0, GP1, GP6 and GP9 are now unused with no-connect flags
- Board pads re-netted from the new netlist (87 pads)

QMK pin lists must follow this map. ERC 0 errors; DRC with schematic
parity shows only the expected unconnected items and starved thermals.
Connections:
- net GP18: now also SW10.1, SW20.1, SW30.1, SW40.1, SW50.1, SW60.1; no longer SW15.1, SW25.1, SW35.1, SW45.1, SW55.1, SW65.1 (SW)
- net GP19: now also SW11.1, SW21.1, SW31.1, SW41.1, SW51.1, SW61.1; no longer SW14.1, SW24.1, SW34.1, SW44.1, SW54.1, SW64.1
- net GP2: now also JP1.2 (C); no longer D40.1, D41.1, D42.1, D43.1, D44.1, D45.1
- net GP21: now also SW13.1, SW23.1, SW33.1, SW43.1, SW53.1, SW63.1; no longer JP1.2 (C)
- net GP22: now also SW14.1, SW24.1, SW34.1, SW44.1, SW54.1, SW64.1; no longer SW65.B
- net GP23: now also SW15.1, SW25.1, SW35.1, SW45.1, SW55.1, SW65.1 (SW); no longer SW65.A
- net GP24: now also D60.1, D61.1, D62.1, D63.1, D64.1, D65.1; no longer SW13.1, SW23.1, SW33.1, SW43.1, SW53.1, SW63.1
- net GP25: now also D50.1, D51.1, D52.1, D53.1, D54.1, D55.1; no longer SW12.1, SW22.1, SW32.1, SW42.1, SW52.1, SW62.1
- net GP26: now also D40.1, D41.1, D42.1, D43.1, D44.1, D45.1; no longer SW11.1, SW21.1, SW31.1, SW41.1, SW51.1, SW61.1
- net GP27: now also D30.1, D31.1, D32.1, D33.1, D34.1, D35.1; no longer SW10.1, SW20.1, SW30.1, SW40.1, SW50.1, SW60.1
- net GP28: now also D20.1, D21.1, D22.1, D23.1, D24.1, D25.1; no longer JP3.1 (A), R12.2
- net GP29: now also D10.1, D11.1, D12.1, D13.1, D14.1, D15.1, D16.1; no longer JP2.1 (A), R13.2
- net GP3: now also SW65.B; no longer D50.1, D51.1, D52.1, D53.1, D54.1, D55.1
- net GP4: now also SW65.A; no longer D60.1, D61.1, D62.1, D63.1, D64.1, D65.1
- net GP16: now reaches U1.27 (GPIO16)
- net GP16: now also JP3.1 (A), R12.2
- net GP17: now reaches U1.28 (GPIO17)
- net GP17: now also JP2.1 (A), R13.2
- net GP20: now reaches U1.31 (GPIO20)
- net GP20: now also SW12.1, SW22.1, SW32.1, SW42.1, SW52.1, SW62.1
- removed net GP0: D20.1, D21.1, D22.1, D23.1, D24.1, D25.1, U1.2 (GPIO0)
- removed net GP1: D30.1, D31.1, D32.1, D33.1, D34.1, D35.1, U1.3 (GPIO1)
- removed net GP6: D10.1, D11.1, D12.1, D13.1, D14.1, D15.1, D16.1, U1.8 (GPIO6)

Commit message: feat(pcb): swap row and column pins and clear u1's trunk side
Rows now leave U1 on the west-facing pins and columns on the north-west
pins, so each group heads straight for its corridor. A few parts moved
off U1's matrix side for the same reason.

- Rows 1-6 on GP23-GP18 (pins 35-29), columns 0-5 on GP29-GP24
  (pins 41-36); the encoder-key column stays on GP5
- R10/R11 moved next to GP13, C13/C14 off the west and north-west pins,
  F1 moved clear of the F.Cu trunk corridor left of the strip

ERC 0 errors; DRC with schematic parity shows only unconnected items
and starved thermals (the board is still unrouted).
Connections:
- net GP18: now also D60.1, D61.1, D62.1, D63.1, D64.1, D65.1; no longer SW10.1, SW20.1, SW30.1, SW40.1, SW50.1, SW60.1
- net GP19: now also D50.1, D51.1, D52.1, D53.1, D54.1, D55.1; no longer SW11.1, SW21.1, SW31.1, SW41.1, SW51.1, SW61.1
- net GP20: now also D40.1, D41.1, D42.1, D43.1, D44.1, D45.1; no longer SW12.1, SW22.1, SW32.1, SW42.1, SW52.1, SW62.1
- net GP21: now also D30.1, D31.1, D32.1, D33.1, D34.1, D35.1; no longer SW13.1, SW23.1, SW33.1, SW43.1, SW53.1, SW63.1
- net GP22: now also D20.1, D21.1, D22.1, D23.1, D24.1, D25.1; no longer SW14.1, SW24.1, SW34.1, SW44.1, SW54.1, SW64.1
- net GP23: now also D10.1, D11.1, D12.1, D13.1, D14.1, D15.1, D16.1; no longer SW15.1, SW25.1, SW35.1, SW45.1, SW55.1, SW65.1 (SW)
- net GP24: now also SW15.1, SW25.1, SW35.1, SW45.1, SW55.1, SW65.1 (SW); no longer D60.1, D61.1, D62.1, D63.1, D64.1, D65.1
- net GP25: now also SW14.1, SW24.1, SW34.1, SW44.1, SW54.1, SW64.1; no longer D50.1, D51.1, D52.1, D53.1, D54.1, D55.1
- net GP26: now also SW13.1, SW23.1, SW33.1, SW43.1, SW53.1, SW63.1; no longer D40.1, D41.1, D42.1, D43.1, D44.1, D45.1
- net GP27: now also SW12.1, SW22.1, SW32.1, SW42.1, SW52.1, SW62.1; no longer D30.1, D31.1, D32.1, D33.1, D34.1, D35.1
- net GP28: now also SW11.1, SW21.1, SW31.1, SW41.1, SW51.1, SW61.1; no longer D20.1, D21.1, D22.1, D23.1, D24.1, D25.1
- net GP29: now also SW10.1, SW20.1, SW30.1, SW40.1, SW50.1, SW60.1; no longer D10.1, D11.1, D12.1, D13.1, D14.1, D15.1, D16.1

Commit message: feat(pcb): move to 4 layers with planes, wson flash and usb pairs
Applies the accepted v5e controller placement and turns the board into a
4-layer design, so the controller strip has room to be hand routed and the
USB lines get a proper reference.

- U1 straight at 180 degrees and 4 mm lower, every signal pin keeping a
  3.5 mm escape lane; caps, crystal and flash follow the RP2040 Community
  Edition controllers
- 16 MB flash swapped to the WSON W25Q128JVPIQ (LCSC C190862), which halves
  the QSPI run to 25.7 mm
- inner GND and +5V planes with a +3.3V island under the controller, and no
  plane under the crystal
- USB data renamed into real pairs (D_USB, USB_MCU, LINK_D) with a rule that
  holds each pair to 0.1 mm length match and keeps it coupled

ERC 0 errors. DRC: no schematic parity issues, only unconnected items and
starved thermals, since the board carries no tracks yet.
Parts:
- U3: footprint PCM_JLCPCB:SOIC-8_L5.3-W5.3-P1.27-LS8.0-BL -> Package_SON:WSON-8-1EP_6x5mm_P1.27mm_EP3.4x4mm; LCSC C97521 -> C190862; Part W25Q128JVSIQ -> W25Q128JVPIQ
Connections:
- net USB_MCU_P: now reaches R7.2, U1.47 (USB_DP)
- net USB_MCU_N: now reaches R8.2, U1.46 (USB_DM)
- net LINK_DATA renamed LINK_D_P
- net SPLIT_D_N renamed LINK_D_N
Changed lines of the file:
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@@
 		)
 	)
-	(global_label "LINK_DATA"
+	(global_label "LINK_D_P"
 		(shape input)
 		(at 69.85 271.78 0)
@@
 		)
 	)
-	(global_label "LINK_DATA"
+	(global_label "LINK_D_P"
 		(shape input)
 		(at 127 269.24 0)
@@
 		)
 	)
-	(global_label "SPLIT_D_N"
+	(global_label "LINK_D_N"
 		(shape input)
 		(at 33.02 261.62 180)
@@
 		)
 	)
-	(global_label "SPLIT_D_N"
+	(global_label "LINK_D_N"
 		(shape input)
 		(at 127 264.16 0)
@@
 		)
 	)
-	(global_label "LINK_DATA"
+	(global_label "LINK_D_P"
 		(shape input)
 		(at 156.21 280.67 180)
@@
 		)
 	)
+	(global_label "USB_MCU_N"
+		(shape input)
+		(at 161.29 92.71 180)
+		(fields_autoplaced yes)
+		(effects
+			(font
+				(size 1.27 1.27)
+			)
+			(justify left)
+		)
+		(property "Intersheetrefs" "${INTERSHEET_REFS}"
+			(at 169.234 92.71 0)
+			(hide yes)
+			(show_name no)
+			(do_not_autoplace no)
+			(effects
+				(font
+					(size 1.27 1.27)
+				)
+				(justify left)
+			)
+		)
+	)
+	(global_label "USB_MCU_P"
+		(shape input)
+		(at 161.29 90.17 180)
+		(fields_autoplaced yes)
+		(effects
+			(font
+				(size 1.27 1.27)
+			)
+			(justify left)
+		)
+		(property "Intersheetrefs" "${INTERSHEET_REFS}"
+			(at 169.234 90.17 0)
+			(hide yes)
+			(show_name no)
+			(do_not_autoplace no)
+			(effects
+				(font
+					(size 1.27 1.27)
+				)
+				(justify left)
+			)
+		)
+	)
 	(symbol
 		(lib_id "power:+3.3V")
@@
 			)
 		)
-		(property "Footprint" "PCM_JLCPCB:SOIC-8_L5.3-W5.3-P1.27-LS8.0-BL"
+		(property "Footprint" "Package_SON:WSON-8-1EP_6x5mm_P1.27mm_EP3.4x4mm"
 			(at 55.88 181.61 0)
 			(hide yes)
@@
 			)
 		)
-		(property "Datasheet" "https://www.lcsc.com/datasheet/lcsc_datasheet_1811142111_Winbond-Elec-W25Q128JVSIQ_C97521.pdf"
+		(property "Datasheet" "https://www.lcsc.com/datasheet/lcsc_datasheet_1811151432_Winbond-Elec-W25Q128JVPIQ_C190862.pdf"
 			(at 53.594 171.323 0)
 			(hide yes)
@@
 			)
 		)
-		(property "LCSC" "C97521"
+		(property "LCSC" "C190862"
 			(at 55.88 171.45 0)
 			(hide yes)
@@
 			)
 		)
-		(property "Part" "W25Q128JVSIQ"
+		(property "Part" "W25Q128JVPIQ"
 			(at 55.88 171.45 0)
 			(hide yes)

Commit message: feat(pcb): swap usb-c and esd parts, fix nets, rules and silkscreen
Moves both USB-C ports to the part every reference board uses, shrinks the
ESD arrays and cleans up the nets, rules and silkscreen around them. The
board passes ERC and DRC with no errors and no schematic parity issues.

- USB-C J1/J2 are now HRO TYPE-C-31-M-12 (LCSC C165948), the connector the
  RP2040 design guide, Corne v4, Djinn, Ferris and sea-picro all use, with
  its real 3D model and a project footprint whose pad numbers match our
  symbol; both sit 0.49 mm proud of the board edge, per its datasheet
- ESD arrays are USBLC6-2P6 in SOT-563 (2.0 x 2.5 mm against 3.1 x 2.1),
  and their two channels now carry each data line through the part, which
  is the layout ST and TI ask for
- USB nets are named per segment so each side of R7/R8 is its own net:
  D+/D- from the connector, USB_P/USB_N into the MCU
- R7/R8 moved 12.7 mm clear of U1 so the MCU-side labels have a wire to sit
  on instead of printing over the chip symbol
- protection parts sit at the connectors: fuse 2.5 mm from the 5 V pad,
  ESD 1.5 to 2.0 mm from the data pads, diode right after the fuse
- fuses raised to 1.1 A (LCSC C126818): 37 LEDs at the planned brightness
  draw about 0.8 A through one half's fuse, which would trip a 500 mA part

Under the hood:

- design rules follow JLCPCB's published limits: 0.3 mm copper to edge,
  0.4 mm minimum via, 0.15 mm silkscreen lines and 1.0 mm text
- one diff pair rule per pair, with spacing checked outside the fan-out and
  length across the whole net; a shared rule compared nets across ports,
  and a rule condition split over two lines was silently ignored
- no pair rule on the link port: it is one-wire serial, and LINK_D_N never
  reaches the MCU
- GND plane moved to the inner layer next to the parts, so USB, ESD and
  decoupling reference solid ground
- crystal keep-out now covers the power plane only: Abracon and Raspberry
  Pi ask for short traces, not cleared ground, and the plane a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
Parts:
- F1, F2: value 500mA -> 1.1A; LCSC C163512 -> C126818; Part 1206L050YR -> 1206L110THYR
- J1, J2: footprint PCM_JLCPCB:TYPE-C-SMD_HX-TYPE-C-16PIN -> my-soffle:USB_C_Receptacle_HRO_TYPE-C-31-M-12_MergedPads; LCSC C2927039 -> C165948
- U2, U4: value SRV05-4 -> USBLC6-2P6; footprint PCM_JLCPCB:SOT-23-6_L2.9-W1.6-P0.95-LS2.9-BL -> Package_TO_SOT_SMD:SOT-563; symbol PCM_JLCPCB-Diode-Packages:Package, SRV05-4A_C20615829 -> Power_Protection:USBLC6-2P6; LCSC C2836319 -> C49451919
- U3: value W25Q128 -> W25Q128JVPIQ
Connections:
- net LINK_D_N: now also U2.3 (I/O2)
- net LINK_D_P: now also U2.6 (I/O1)
- net D-: now reaches U4.3 (I/O2)
- net D-: now also J1.A7 (D-), J1.B7 (D-), R8.1, U4.4 (I/O2)
- removed net D_USB_N: J1.A7 (D-), J1.B7 (D-), R8.1, U4.6 (I/O)
- net D_USB_P renamed D+
- net D+: now also U4.6 (I/O1)
- net USB_MCU_N renamed USB_N
- net USB_MCU_P renamed USB_P
- no-connect marks 18 -> 14
Other:
- moved on the sheet: R7, R8
