File: sofle-choc-pro.kicad_sch (KiCad schematic)
At the start: 194 parts, among them J1 Connector, USB-TYPE-C-16P, J2 Connector, USB-TYPE-C-16P, J3 OLED 128x32, SW1 BOOT, SW10 F0, SW11 F1, SW12 F2, SW13 F3, SW14 F4, SW15 F5, SW16 F6 Choc/EC11, SW2 RESET, SW20 N0, SW21 N1, SW22 N2, SW23 N3, SW24 N4, SW25 N5, SW30 T0, SW31 T1, SW32 T2, SW33 T3, SW34 T4, SW35 T5, SW40 H0, SW41 H1, SW42 H2, SW43 H3, SW44 H4, SW45 H5, SW50 B0, SW51 B1, SW52 B2, SW53 B3, SW54 B4, SW55 B5, SW60 TH0, SW61 TH1, SW62 TH2, SW63 TH3, SW64 TH4, SW65 TH5 Choc/EC11, U1 RP2040, U2 USBLC6-2P6, U3 W25Q128JVPIQ, U4 USBLC6-2P6, U5 AP2112K-3.3, U6 SN74LV1T34DBVR, X1 ABM8-272-T3

Commit message: feat(pcb): move both halves to a mid-mount usb-c
Both USB-C connectors on both halves move from the HRO TYPE-C-31-M-12
top-mount part to Hong Cheng's HC-TYPE-C-16P-C16B, which sinks 1.60 mm
into the board. On a 1.6 mm PCB that leaves nothing hanging underneath,
which is what takes the connector out of the standoff budget and lets
the case stack reach 8.2 mm. This commit also carries the earlier strip
of signal routing on both halves, leaving power only, so they can be
hand routed from scratch.

- J1 and J2 sit 0.785 mm closer to their board edges, because the new
  body is 6.50 mm deep against the old 7.35, so the port still meets
  the edge
- The board outline gains a 9.24 x 5.75 mm cutout at each port
- The spacer is pocketed over each connector body, which now stands
  1.66 mm proud of the board top instead of hanging below it
- C10 and C11 move 0.7 mm north, with their 3.3 V feeds and island
  vias, clear of J2's wider shell legs

Under the hood:
- lib: new footprint measured off the manufacturer drawing rather than
  taken from the EasyEDA model, which puts the shell holes 11.25 mm
  apart instead of 10.79 and cuts the slot 6.40 mm deep instead of 5.75
- ergogen: usbc_sink and usbc_above replace a symmetric mid-mount guess
  that had the body straddling the board; board_pcb subtracts the port
  slots so the case and plate outlines keep their walls
- dru: "usb-c land to cutout" allows the 0.15 mm the drawing specifies,
  scoped to J1/J2 pads so other copper keeps the 0.3 mm rule

ERC 0 and schematic parity 0 on both halves. DRC is down to the 13
pre-existing mounting hole courtyard overlaps per board. JLCPCB quote
0.3 mm copper to a routed outline, so the 0.15 mm lands may draw a
query on the first order.
Parts:
- J1, J2: footprint my-soffle:USB_C_Receptacle_HRO_TYPE-C-31-M-12_MergedPads -> my-soffle:USB_C_Receptacle_HongCheng_HC-TYPE-C-16P_MidMount; LCSC C165948 -> C19274022
Changed lines of the file:
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@@
 			)
 		)
-		(property "Footprint" "my-soffle:USB_C_Receptacle_HRO_TYPE-C-31-M-12_MergedPads"
+		(property "Footprint" "my-soffle:USB_C_Receptacle_HongCheng_HC-TYPE-C-16P_MidMount"
 			(at 26.67 50.8 0)
 			(hide yes)
@@
 			)
 		)
-		(property "Datasheet" "https://jlcpcb.com/partdetail/Korean_HropartsElec-TYPE_C_31_M12/C165948"
+		(property "Datasheet" "https://www.lcsc.com/product-detail/C19274022.html"
 			(at 24.384 40.513 0)
 			(hide yes)
@@
 			)
 		)
-		(property "LCSC" "C165948"
+		(property "LCSC" "C19274022"
 			(at 29.21 39.37 0)
 			(hide yes)
@@
 			)
 		)
-		(property "Footprint" "my-soffle:USB_C_Receptacle_HRO_TYPE-C-31-M-12_MergedPads"
+		(property "Footprint" "my-soffle:USB_C_Receptacle_HongCheng_HC-TYPE-C-16P_MidMount"
 			(at 106.68 283.21 0)
 			(hide yes)
@@
 			)
 		)
-		(property "Datasheet" "https://jlcpcb.com/partdetail/Korean_HropartsElec-TYPE_C_31_M12/C165948"
+		(property "Datasheet" "https://www.lcsc.com/product-detail/C19274022.html"
 			(at 104.394 272.923 0)
 			(hide yes)
@@
 			)
 		)
-		(property "LCSC" "C165948"
+		(property "LCSC" "C19274022"
 			(at 109.22 271.78 0)
 			(hide yes)

Commit message: feat(pcb): put both halves in one project and one board
Both halves now live in one KiCad project: the schematic is one half sheet
used twice, as sheets Left and Right, and one board carries both halves
10 mm apart, so they are seen, checked and ordered together. Nothing moved
or was rewired: every pad sits where it did on the two old boards and every
pad net matches the new schematic.

- Edit sofle-choc-pro-half.kicad_sch once and both halves follow; Right
  references are the Left ones + 200
- Every net is per half, power included, through local power symbols, so
  the two halves can never join into one net
- One Ergogen run builds both halves, and the USB-C notches, case ports,
  spacer pockets and display openings hang off J1-J3 points, so board and
  case cannot drift apart
- Placement, LED snapping and hole placement work on both halves by
  (half, role)

Under the hood:
- sch: global labels made local; VBUS_FUSED names the F1-D1 net, which
  only had an auto name; H1-H5 are MountingHole symbols now
- pcb: right board brought in +139 mm with fresh UUIDs; its 29 unplaced
  support parts parked below it; pours clipped at the midline; J1/J2
  origins moved onto the board edge; the right HOST/LINK labels mirrored
  from the left, since they were stale copies at the left's coordinates
- rules: net class patterns and pair rules use sheet-prefixed names, which
  bare names never match; one skew rule per half so the pairs are not
  compared across halves
- ergogen: make_right.js becomes make_both.js; mounts.json replaces
  screws.json
- scripts: halves.py added; place_mounting_holes.py folded into
  place_from_ergogen.py; strip_signals.py keeps VBUS_FUSED as power
- fixes: the holes and J1/J2 had bare footprint ids or no sheet fields

ERC 0, parity 0, 452 unconnected (194 + 258, unrouted). DRC errors are the
26 known hole courtyard overlaps, 13 per half.
Parts:
- removed C1, C4: 15pF, PCM_JLCPCB:C_0402, symbol PCM_JLCPCB-Capacitors:0402,15pF
- removed C10, C11, C110, C111, C112, C113, C114, C115, C116, C12, C120, C121, C122, C123, C124, C125, C13, C130, C131, C132, C133, C134, C135, C14, C140, C141, C142, C143, C144, C145, C15, C150, C151, C152, C153, C154, C155, C16, C160, C161, C162, C163, C164, C165, C17, C3, C30, C5, C6: 100nF, PCM_JLCPCB:C_0402, symbol PCM_JLCPCB-Capacitors:0402,100nF
- removed C18, C9: 10uF, PCM_JLCPCB:C_0603, symbol PCM_JLCPCB-Capacitors:0603,10uF
- removed C19, C20, C7, C8: 1uF, PCM_JLCPCB:C_0402, symbol PCM_JLCPCB-Capacitors:0402,1uF
- removed D1: B5819W SL, PCM_JLCPCB:D_SOD-123, symbol PCM_JLCPCB-Diodes:Schottky,B5819W SL
- removed D10, D11, D12, D13, D14, D15, D16, D20, D21, D22, D23, D24, D25, D30, D31, D32, D33, D34, D35, D40, D41, D42, D43, D44, D45, D50, D51, D52, D53, D54, D55, D60, D61, D62, D63, D64, D65: 1N4148W, PCM_JLCPCB:D_SOD-123, symbol PCM_JLCPCB-Diodes:Switching,1N4148W
- removed F1, F2: 1.1A, Fuse:Fuse_1206_3216Metric, symbol Device:Polyfuse
- removed J1, J2: Connector, USB-TYPE-C-16P, my-soffle:USB_C_Receptacle_HongCheng_HC-TYPE-C-16P_MidMount, symbol PCM_JLCPCB-Extended:Connector, USB-TYPE-C-16P
- removed J3: OLED 128x32, Connector_PinHeader_2.54mm:PinHeader_1x04_P2.54mm_Vertical, symbol Connector_Generic:Conn_01x04
- removed JP1: HAND L=1-2 R=2-3, Jumper:SolderJumper-3_P1.3mm_Open_RoundedPad1.0x1.5mm_NumberLabels, symbol Jumper:SolderJumper_3_Open
- removed LED10, LED11, LED12, LED13, LED14, LED15, LED16, LED20, LED21, LED22, LED23, LED24, LED25, LED30, LED31, LED32, LED33, LED34, LED35, LED40, LED41, LED42, LED43, LED44, LED45, LED50, LED51, LED52, LED53, LED54, LED55, LED60, LED61, LED62, LED63, LED64, LED65: SK6812MINI-E, my-soffle:LED-SMD_4P-L3.2-W2.8-LS5.9_SK6812MINI-E, symbol my-soffle:SK6812MINI-E_C5149201
- removed R10, R11: 10kΩ, PCM_JLCPCB:R_0402, symbol PCM_JLCPCB-Resistors:0402,10kΩ
- removed R15: 470Ω, PCM_JLCPCB:R_0402, symbol PCM_JLCPCB-Resistors:0402,470Ω
- removed R16: 120Ω, PCM_JLCPCB:R_0402, symbol PCM_JLCPCB-Resistors:0402,120Ω
- removed R2, R4: 1kΩ, PCM_JLCPCB:R_0402, symbol PCM_JLCPCB-Resistors:0402,1kΩ
- removed R5, R6: 5.1kΩ, PCM_JLCPCB:R_0402, symbol PCM_JLCPCB-Resistors:0402,5.1kΩ
- removed R7, R8: 27Ω, PCM_JLCPCB:R_0402, symbol PCM_JLCPCB-Resistors:0402,33Ω
- removed SW1: BOOT, my-soffle:SW_Push_1P1T_XUNPU_TS-1088-AR02016, symbol Switch:SW_Push
- removed SW10: F0, my-soffle:SW_Choc_V1V2_Hotswap_1.00u, symbol Switch:SW_Push
- removed SW11: F1, my-soffle:SW_Choc_V1V2_Hotswap_1.00u, symbol Switch:SW_Push
- removed SW12: F2, my-soffle:SW_Choc_V1V2_Hotswap_1.00u, symbol Switch:SW_Push
- removed SW13: F3, my-soffle:SW_Choc_V1V2_Hotswap_1.00u, symbol Switch:SW_Push
- removed SW14: F4, my-soffle:SW_Choc_V1V2_Hotswap_1.00u, symbol Switch:SW_Push
- removed SW15: F5, my-soffle:SW_Choc_V1V2_Hotswap_1.00u, symbol Switch:SW_Push
- removed SW16: F6 Choc/EC11, my-soffle:SW_Choc_V1V2_Hotswap_EC11_Combo, symbol my-soffle:SW_Choc_EC11_Combo
- removed SW2: RESET, my-soffle:SW_Push_1P1T_XUNPU_TS-1088-AR02016, symbol Switch:SW_Push
- removed SW20: N0, my-soffle:SW_Choc_V1V2_Hotswap_1.00u, symbol Switch:SW_Push
- removed SW21: N1, my-soffle:SW_Choc_V1V2_Hotswap_1.00u, symbol Switch:SW_Push
- removed SW22: N2, my-soffle:SW_Choc_V1V2_Hotswap_1.00u, symbol Switch:SW_Push
- removed SW23: N3, my-soffle:SW_Choc_V1V2_Hotswap_1.00u, symbol Switch:SW_Push
- removed SW24: N4, my-soffle:SW_Choc_V1V2_Hotswap_1.00u, symbol Switch:SW_Push
- removed SW25: N5, my-soffle:SW_Choc_V1V2_Hotswap_1.00u, symbol Switch:SW_Push
- removed SW30: T0, my-soffle:SW_Choc_V1V2_Hotswap_1.00u, symbol Switch:SW_Push
- removed SW31: T1, my-soffle:SW_Choc_V1V2_Hotswap_1.00u, symbol Switch:SW_Push
- removed SW32: T2, my-soffle:SW_Choc_V1V2_Hotswap_1.00u, symbol Switch:SW_Push
- removed SW33: T3, my-soffle:SW_Choc_V1V2_Hotswap_1.00u, symbol Switch:SW_Push
- removed SW34: T4, my-soffle:SW_Choc_V1V2_Hotswap_1.00u, symbol Switch:SW_Push
- removed SW35: T5, my-soffle:SW_Choc_V1V2_Hotswap_1.00u, symbol Switch:SW_Push
- removed SW40: H0, my-soffle:SW_Choc_V1V2_Hotswap_1.00u, symbol Switch:SW_Push
- removed SW41: H1, my-soffle:SW_Choc_V1V2_Hotswap_1.00u, symbol Switch:SW_Push
- removed SW42: H2, my-soffle:SW_Choc_V1V2_Hotswap_1.00u, symbol Switch:SW_Push
- removed SW43: H3, my-soffle:SW_Choc_V1V2_Hotswap_1.00u, symbol Switch:SW_Push
- removed SW44: H4, my-soffle:SW_Choc_V1V2_Hotswap_1.00u, symbol Switch:SW_Push
- removed SW45: H5, my-soffle:SW_Choc_V1V2_Hotswap_1.00u, symbol Switch:SW_Push
- removed SW50: B0, my-soffle:SW_Choc_V1V2_Hotswap_1.00u, symbol Switch:SW_Push
- removed SW51: B1, my-soffle:SW_Choc_V1V2_Hotswap_1.00u, symbol Switch:SW_Push
- removed SW52: B2, my-soffle:SW_Choc_V1V2_Hotswap_1.00u, symbol Switch:SW_Push
- removed SW53: B3, my-soffle:SW_Choc_V1V2_Hotswap_1.00u, symbol Switch:SW_Push
- removed SW54: B4, my-soffle:SW_Choc_V1V2_Hotswap_1.00u, symbol Switch:SW_Push
- removed SW55: B5, my-soffle:SW_Choc_V1V2_Hotswap_1.00u, symbol Switch:SW_Push
- removed SW60: TH0, my-soffle:SW_Choc_V1V2_Hotswap_1.00u, symbol Switch:SW_Push
- removed SW61: TH1, my-soffle:SW_Choc_V1V2_Hotswap_1.00u, symbol Switch:SW_Push
- removed SW62: TH2, my-soffle:SW_Choc_V1V2_Hotswap_1.00u, symbol Switch:SW_Push
- removed SW63: TH3, my-soffle:SW_Choc_V1V2_Hotswap_1.00u, symbol Switch:SW_Push
- removed SW64: TH4, my-soffle:SW_Choc_V1V2_Hotswap_1.50u, symbol Switch:SW_Push
- removed SW65: TH5 Choc/EC11, my-soffle:SW_Choc_V1V2_Hotswap_EC11_Combo, symbol my-soffle:SW_Choc_EC11_Combo
- removed U1: RP2040, PCM_JLCPCB:QFN-56-1EP_7x7mm_P0.4mm_EP3.2x3.2mm_ThermalVias, symbol PCM_JLCPCB-Extended:MCU, RP2040
- removed U2, U4: USBLC6-2P6, my-soffle:SOT-563_USBLC6-2P6, symbol Power_Protection:USBLC6-2P6
- removed U3: W25Q128JVPIQ, Package_SON:WSON-8-1EP_6x5mm_P1.27mm_EP3.4x4mm, symbol PCM_JLCPCB-Memory:16MByte, SPI
- removed U5: AP2112K-3.3, PCM_JLCPCB:SOT-23-5_L3.0-W1.7-P0.95-LS2.8-BL, symbol Regulator_Linear:AP2112K-3.3
- removed U6: SN74LV1T34DBVR, Package_TO_SOT_SMD:SOT-23-5, symbol 74xGxx:74LVC1G34
- removed X1: ABM8-272-T3, PCM_JLCPCB:CRYSTAL-SMD_4P-L3.2-W2.5-BL, symbol PCM_JLCPCB-Crystals:Crystal, 12MHz, 20pF
Connections:
- no-connect marks 18 -> 0
Other:
- added sheet Left (sofle-choc-pro-half.kicad_sch)
- added sheet Right (sofle-choc-pro-half.kicad_sch)
- note removed: "12MHZ-CRYSTAL"
- note removed: "16MB-FLASH"
- note removed: "DECOUPLING CAPACITORS"
- note removed: "ESD PROTECTION HOST"
- note removed: "ESD PROTECTION INTERCONNECT"
- note removed: "USB-C INTERCONNECT"
- note removed: "USB-C-16P-2A + FUSE LDO-5V-->3V3"
