File: sofle-choc-pro-right.kicad_pcb (KiCad board)
At the start: 4 copper layers, 129 x 118 mm, 199 parts, among them J1 Connector, USB-TYPE-C-16P, J2 Connector, USB-TYPE-C-16P, J3 OLED 128x32, SW1 BOOT, SW10 F0, SW11 F1, SW12 F2, SW13 F3, SW14 F4, SW15 F5, SW16 F6 Choc/EC11, SW2 RESET, SW20 N0, SW21 N1, SW22 N2, SW23 N3, SW24 N4, SW25 N5, SW30 T0, SW31 T1, SW32 T2, SW33 T3, SW34 T4, SW35 T5, SW40 H0, SW41 H1, SW42 H2, SW43 H3, SW44 H4, SW45 H5, SW50 B0, SW51 B1, SW52 B2, SW53 B3, SW54 B4, SW55 B5, SW60 TH0, SW61 TH1, SW62 TH2, SW63 TH3, SW64 TH4, SW65 TH5 Choc/EC11, U1 RP2040, U2 USBLC6-2P6, U3 W25Q128JVPIQ, U4 USBLC6-2P6, U5 AP2112K-3.3, U6 SN74LV1T34DBVR, X1 ABM8-272-T3

Commit message: feat(pcb): move both halves to a mid-mount usb-c
Both USB-C connectors on both halves move from the HRO TYPE-C-31-M-12
top-mount part to Hong Cheng's HC-TYPE-C-16P-C16B, which sinks 1.60 mm
into the board. On a 1.6 mm PCB that leaves nothing hanging underneath,
which is what takes the connector out of the standoff budget and lets
the case stack reach 8.2 mm. This commit also carries the earlier strip
of signal routing on both halves, leaving power only, so they can be
hand routed from scratch.

- J1 and J2 sit 0.785 mm closer to their board edges, because the new
  body is 6.50 mm deep against the old 7.35, so the port still meets
  the edge
- The board outline gains a 9.24 x 5.75 mm cutout at each port
- The spacer is pocketed over each connector body, which now stands
  1.66 mm proud of the board top instead of hanging below it
- C10 and C11 move 0.7 mm north, with their 3.3 V feeds and island
  vias, clear of J2's wider shell legs

Under the hood:
- lib: new footprint measured off the manufacturer drawing rather than
  taken from the EasyEDA model, which puts the shell holes 11.25 mm
  apart instead of 10.79 and cuts the slot 6.40 mm deep instead of 5.75
- ergogen: usbc_sink and usbc_above replace a symmetric mid-mount guess
  that had the body straddling the board; board_pcb subtracts the port
  slots so the case and plate outlines keep their walls
- dru: "usb-c land to cutout" allows the 0.15 mm the drawing specifies,
  scoped to J1/J2 pads so other copper keeps the 0.3 mm rule

ERC 0 and schematic parity 0 on both halves. DRC is down to the 13
pre-existing mounting hole courtyard overlaps per board. JLCPCB quote
0.3 mm copper to a routed outline, so the 0.15 mm lands may draw a
query on the first order.
Parts:
- J1, J2: footprint my-soffle:USB_C_Receptacle_HRO_TYPE-C-31-M-12_MergedPads -> my-soffle:USB_C_Receptacle_HongCheng_HC-TYPE-C-16P_MidMount
- moved J1 0.79 mm to (59.2, 63.8)
- moved J2 0.78 mm to (51.9, 93.7)
Routing:
- net Net-(D65-Pad2): track 16.2 -> 0.00 mm
- net Net-(D16-Pad2): track 15.6 -> 0.00 mm
- net SS: track 13.0 -> 0.00 mm
- net SD1: track 11.2 -> 0.00 mm
- net SD2: track 9.73 -> 0.00 mm
- net SD3: track 7.13 -> 0.00 mm
- net CLK: track 5.96 -> 0.00 mm
- net Net-(D63-Pad2): track 5.32 -> 0.00 mm
- net Net-(D64-Pad2): track 4.54 -> 0.00 mm
- net Net-(D62-Pad2): track 4.52 -> 0.00 mm
- net Net-(D61-Pad2): track 4.52 -> 0.00 mm
- net Net-(D60-Pad2): track 4.52 -> 0.00 mm
- net Net-(D55-Pad2): track 4.52 -> 0.00 mm
- net Net-(D54-Pad2): track 4.52 -> 0.00 mm
- net Net-(D53-Pad2): track 4.52 -> 0.00 mm
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Other:
- outline, holes or cut-outs redrawn
