File: velvet74-half.kicad_sch (KiCad schematic)
At the start: 200 parts, among them J1 Connector, USB-TYPE-C-16P, J2 Connector, USB-TYPE-C-16P, J3 OLED 128x32, SW1 BOOT, SW10 F0, SW11 F1, SW12 F2, SW13 F3, SW14 F4, SW15 F5, SW16 F6 Choc/EC11, SW2 RESET, SW20 N0, SW21 N1, SW22 N2, SW23 N3, SW24 N4, SW25 N5, SW30 T0, SW31 T1, SW32 T2, SW33 T3, SW34 T4, SW35 T5, SW40 H0, SW41 H1, SW42 H2, SW43 H3, SW44 H4, SW45 H5, SW50 B0, SW51 B1, SW52 B2, SW53 B3, SW54 B4, SW55 B5, SW60 TH0, SW61 TH1, SW62 TH2, SW63 TH3, SW64 TH4, SW65 TH5 Choc/EC11, U1 RP2040, U2 USBLC6-2P6, U3 ZD25Q128CWIGR, U4 USBLC6-2P6, U5 AP2112K-3.3, U6 SN74LV1T34DBVR, X1 ABM8-272-T3

Commit message: docs(kicad): fill the title blocks
The schematic sheets and the board now carry a title block, so printed
drawings and PDFs say what the board is and which revision.

- Title Velvet74 (the half sheet names both Left and Right), date
  2026-09-23, revision 1.0, company unseensnick
- Comments: what the keyboard is, the panel and stackup, the tools, and
  the repo link

ERC 0. DRC with parity unchanged: 42 known items, 0 unconnected,
0 parity.
Other:
- company: (none) -> unseensnick
- title: (none) -> Velvet74 half (sheets Left and Right)
Changed lines of the file:
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@@
 	(generator_version "10.0")
 	(paper "E")
+	(title_block
+		(title "Velvet74 half (sheets Left and Right)")
+		(date "2026-09-23")
+		(rev "1.0")
+		(company "unseensnick")
+		(comment 1 "Split Choc keyboard, 74 keys, chip-down RP2040 in each half")
+		(comment 2 "Both halves on one panel, 4-layer 1.6 mm, assembled by JLCPCB")
+		(comment 3 "Key geometry from Ergogen 4.2.1, drawn in KiCad 10.0.3")
+		(comment 4 "github.com/unseensnick/Velvet74")
+	)
 	(rectangle
 		(start 13.97 12.7)
