File: velvet74.kicad_sch (KiCad schematic)
At the start: 0 parts

Commit message: docs(kicad): fill the title blocks
The schematic sheets and the board now carry a title block, so printed
drawings and PDFs say what the board is and which revision.

- Title Velvet74 (the half sheet names both Left and Right), date
  2026-09-23, revision 1.0, company unseensnick
- Comments: what the keyboard is, the panel and stackup, the tools, and
  the repo link

ERC 0. DRC with parity unchanged: 42 known items, 0 unconnected,
0 parity.
Other:
- company: (none) -> unseensnick
- title: (none) -> Velvet74
Changed lines of the file:
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@@
 	(generator_version "10.0")
 	(paper "A4")
+	(title_block
+		(title "Velvet74")
+		(date "2026-09-23")
+		(rev "1.0")
+		(company "unseensnick")
+		(comment 1 "Split Choc keyboard, 74 keys, chip-down RP2040 in each half")
+		(comment 2 "Both halves on one panel, 4-layer 1.6 mm, assembled by JLCPCB")
+		(comment 3 "Key geometry from Ergogen 4.2.1, drawn in KiCad 10.0.3")
+		(comment 4 "github.com/unseensnick/Velvet74")
+	)
 	(sheet
 		(at 40 40)
