File: velvet74.kicad_pcb (KiCad board)
At the start: 4 copper layers, 268 x 133.2 mm, 415 parts, among them J1 Connector, USB-TYPE-C-16P, J2 Connector, USB-TYPE-C-16P, J201 Connector, USB-TYPE-C-16P, J202 Connector, USB-TYPE-C-16P, J203 OLED 128x32, J3 OLED 128x32, SW1 BOOT, SW10 F0, SW11 F1, SW12 F2, SW13 F3, SW14 F4, SW15 F5, SW16 F6 Choc/EC11, SW2 RESET, SW20 N0, SW201 BOOT, SW202 RESET, SW21 N1, SW210 F0, SW211 F1, SW212 F2, SW213 F3, SW214 F4, SW215 F5, SW216 F6 Choc/EC11, SW22 N2, SW220 N0, SW221 N1, SW222 N2, SW223 N3, SW224 N4, SW225 N5, SW23 N3, SW230 T0, SW231 T1, SW232 T2, SW233 T3, SW234 T4, SW235 T5, SW24 N4, SW240 H0, SW241 H1, SW242 H2, SW243 H3, SW244 H4, SW245 H5, SW25 N5, SW250 B0, SW251 B1, SW252 B2, SW253 B3, SW254 B4, SW255 B5, SW260 TH0, SW261 TH1, SW262 TH2, SW263 TH3, SW264 TH4, SW265 TH5 Choc/EC11, SW30 T0, SW31 T1, SW32 T2, SW33 T3, SW34 T4, SW35 T5, SW40 H0, SW41 H1, SW42 H2, SW43 H3, SW44 H4, SW45 H5, SW50 B0, SW51 B1, SW52 B2, SW53 B3, SW54 B4, SW55 B5, SW60 TH0, SW61 TH1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

Commit message: fix(pcb): drop the stale link silkscreen labels
The two LINK labels on the back silkscreen still marked where the link
USB-C used to be, so they pointed at nothing after the port moved.

- Removed both labels (left and right); HOST labels stay
- Both production sets regenerated
Other:
- board text removed: "LINK"
Changed lines of the file:
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@@
-		)
-	)
-	(gr_text "LINK"
-		(at 173.2 102.6 0)
-		(layer "B.SilkS")
-		(effects
-			(font
-				(size 1 1)
-				(thickness 0.15)
-			)
-			(justify mirror)
-		)
-	)
-	(gr_text "LINK"
-		(at 193.8 102.6 0)
-		(layer "B.SilkS")
-		(effects
-			(font
-				(size 1 1)
-				(thickness 0.15)
-			)
-			(justify mirror)
 		)
 	)
